File: pcb/time-slider.kicad_pcb (KiCad board)
At the start: 2 copper layers, 393.1 x 67.2 mm, 67 parts, among them IC1 STPIC6D595MTR, IC2 STPIC6D595MTR, IC3 STPIC6D595MTR, IC4 STPIC6D595MTR, IC5 ESP32-SOLO-1, IC6 CP2102-GMR, J1 Conn_01x06_Pin, J2 Barrel_Jack_MountingPin, M1 Stepper_Motor_unipolar_5pin, M2 Stepper_Motor_unipolar_5pin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

Commit message: Everything should be working
Parts:
- removed JP1: SolderJumper_2_Open, Jumper:SolderJumper-2_P1.3mm_Open_RoundedPad1.0x1.5mm
- removed R7, R8: 0R, Resistor_SMD:R_0402_1005Metric
- added R24: 10k, Resistor_SMD:R_0402_1005Metric, F.Cu at (204.2, 51.2)
- added R25: 10k, Resistor_SMD:R_0402_1005Metric, F.Cu at (221.4, 48.2)
- moved R18 1.11 mm to (248.2, 29.6), turned to 180 degrees
- moved C3 0.41 mm to (391.2, 32.2)
- moved C2 0.39 mm to (178.0, 32.9)
- moved C1 0.28 mm to (37.4, 32.8)
- moved C4 0.20 mm to (256.7, 32.2)
Connections:
- C1 pad 1: +5V -> +3.3V
- C2 pad 1: +5V -> +3.3V
- C3 pad 1: +5V -> +3.3V
- C4 pad 1: +5V -> +3.3V
- C9 pad 1: +5VP -> +12V
- D1 pad 1: +5VP -> +12V
- IC1 pad 1: +5V -> +3.3V
- IC1 pad 7: +5V -> +3.3V
- IC2 pad 1: +5V -> +3.3V
- IC2 pad 7: +5V -> +3.3V
- IC3 pad 1: +5V -> +3.3V
- IC3 pad 7: +5V -> +3.3V
- IC4 pad 1: +5V -> +3.3V
- IC4 pad 7: +5V -> +3.3V
- IC5 pad 35: /TXD -> /RXDO
- IC6 pad 26: /TXDO -> /RXD
- J1 pad 1: +5VP -> /VBUS
- J1 pad 3: /TXD -> /RXDO
- J2 pad 1: +5V -> GND
- J2 pad 3: (no net) -> +12V
- M1 pad 1: GND -> +12V
- M1 pad 2: Net-(IC1-DRAIN6) -> Net-(IC1-DRAIN7)
- M1 pad 3: Net-(IC1-DRAIN7) -> Net-(IC1-DRAIN5)
- M1 pad 4: Net-(IC1-DRAIN5) -> Net-(IC1-DRAIN6)
- M2 pad 1: GND -> +12V
- M2 pad 2: Net-(IC1-DRAIN2) -> Net-(IC1-DRAIN3)
- M2 pad 3: Net-(IC1-DRAIN3) -> Net-(IC1-DRAIN1)
- M2 pad 4: Net-(IC1-DRAIN1) -> Net-(IC1-DRAIN2)
- M3 pad 1: GND -> +12V
- M3 pad 2: Net-(IC2-DRAIN2) -> Net-(IC2-DRAIN3)
- M3 pad 3: Net-(IC2-DRAIN3) -> Net-(IC2-DRAIN1)
- M3 pad 4: Net-(IC2-DRAIN1) -> Net-(IC2-DRAIN2)
- M4 pad 1: GND -> +12V
- M4 pad 2: Net-(IC2-DRAIN6) -> Net-(IC2-DRAIN7)
- M4 pad 3: Net-(IC2-DRAIN7) -> Net-(IC2-DRAIN5)
- M4 pad 4: Net-(IC2-DRAIN5) -> Net-(IC2-DRAIN6)
- M5 pad 1: GND -> +12V
- M5 pad 2: Net-(IC3-DRAIN2) -> Net-(IC3-DRAIN3)
- M5 pad 3: Net-(IC3-DRAIN3) -> Net-(IC3-DRAIN1)
- M5 pad 4: Net-(IC3-DRAIN1) -> Net-(IC3-DRAIN2)
- M6 pad 1: GND -> +12V
- M6 pad 2: Net-(IC3-DRAIN6) -> Net-(IC3-DRAIN7)
- M6 pad 3: Net-(IC3-DRAIN7) -> Net-(IC3-DRAIN5)
- M6 pad 4: Net-(IC3-DRAIN5) -> Net-(IC3-DRAIN6)
- M7 pad 1: GND -> +12V
- M7 pad 2: Net-(IC4-DRAIN2) -> Net-(IC4-DRAIN3)
- M7 pad 3: Net-(IC4-DRAIN3) -> Net-(IC4-DRAIN1)
- M7 pad 4: Net-(IC4-DRAIN1) -> Net-(IC4-DRAIN2)
- M8 pad 1: GND -> +12V
- M8 pad 2: Net-(IC4-DRAIN6) -> Net-(IC4-DRAIN7)
- M8 pad 3: Net-(IC4-DRAIN7) -> Net-(IC4-DRAIN5)
- M8 pad 4: Net-(IC4-DRAIN5) -> Net-(IC4-DRAIN6)
- R1 pad 1: +5VP -> +3.3V
- U1 pad 1: unconnected-(U1-3V3-Pad1) -> +3.3V
- U3 pad 3: +5VP -> +12V
Routing:
- net +12V: track 0.00 -> 505.1 mm, vias 0 -> 2
- net +5V: track 501.6 -> 0.00 mm, vias 2 -> 0
- net +3.3V: track 78.4 -> 508.6 mm, vias 4 -> 9
- net +5VP: track 44.9 -> 0.00 mm, vias 1 -> 0
- net /TXD: track 35.4 -> 0.00 mm
- net /RXDO: track 22.7 -> 56.4 mm
- net /TXDO: track 22.9 -> 0.00 mm
- net /RXD: track 36.1 -> 57.6 mm
- net /VBUS: track 60.7 -> 74.0 mm, vias 2 -> 3
- net Net-(IC3-DRAIN3): track 22.8 -> 11.1 mm
- net Net-(IC4-DRAIN3): track 22.0 -> 11.1 mm
- net Net-(IC2-DRAIN3): track 21.8 -> 11.1 mm
- net Net-(IC4-DRAIN6): track 24.3 -> 13.7 mm
- net Net-(IC1-DRAIN3): track 21.5 -> 11.2 mm
- net Net-(IC3-DRAIN6): track 24.5 -> 14.2 mm
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