File: pcb/time-slider.kicad_sch (KiCad schematic)
At the start: 67 parts, among them IC1 STPIC6D595MTR, IC2 STPIC6D595MTR, IC3 STPIC6D595MTR, IC4 STPIC6D595MTR, IC5 ESP32-SOLO-1, IC6 CP2102-GMR, J1 Conn_01x06_Pin, J2 Barrel_Jack_MountingPin, M1 Stepper_Motor_unipolar_5pin, M2 Stepper_Motor_unipolar_5pin, M3 Stepper_Motor_unipolar_5pin, M4 Stepper_Motor_unipolar_5pin, M5 Stepper_Motor_unipolar_5pin, M6 Stepper_Motor_unipolar_5pin, M7 Stepper_Motor_unipolar_5pin, M8 Stepper_Motor_unipolar_5pin, P1 USB_C_Plug_USB2.0, Q1 SS8050-G, Q2 SS8050-G, SW1 SW_Push, SW2 SW_Push, SW3 SW_Push, SW4 SW_Push, U1 ESP32-DevKitC, U3 AMS1117-3.3

Commit message: Everything should be working
Parts:
- removed JP1: SolderJumper_2_Open, Jumper:SolderJumper-2_P1.3mm_Open_RoundedPad1.0x1.5mm, symbol Jumper:SolderJumper_2_Open
- removed R7, R8: 0R, Resistor_SMD:R_0402_1005Metric, symbol Device:R_Small_US
- added R24, R25: 10k, Resistor_SMD:R_0402_1005Metric, symbol Device:R_Small_US
Connections:
- net TXD is gone; now on net RXDO: IC5.35 (TXD0), J1.3 (Pin_3)
- net TXDO is gone; now on net RXD: IC6.26 (TXD)
- net +3.3V: now also C1.1, C2.1, C3.1, C4.1, IC1.1 (VCC), IC1.7 (~{CLR}), IC2.1 (VCC), IC2.7 (~{CLR}), IC3.1 (VCC), IC3.7 (~{CLR}), IC4.1 (VCC), IC4.7 (~{CLR}), R1.1, U1.1 (3V3), R24.1, R25.2
- net +5V: no longer C1.1, C2.1, C3.1, C4.1, IC1.1 (VCC), IC1.7 (~{CLR}), IC2.1 (VCC), IC2.7 (~{CLR}), IC3.1 (VCC), IC3.7 (~{CLR}), IC4.1 (VCC), IC4.7 (~{CLR}), J2.1
- net EN: now also R24.2
- net GND: now also J2.1; no longer J2.MP (MountPin), M1.1, M2.1, M3.1, M4.1, M5.1, M6.1, M7.1, M8.1
- net IO0: now also R25.1
- net VBUS: now also J1.1 (Pin_1)
- net at IC3.12 (DRAIN5): now also M6.3 (-); no longer M6.4
- net at IC3.13 (DRAIN6): now also M6.4; no longer M6.2
- net at IC3.14 (DRAIN7): now also M6.2; no longer M6.3 (-)
- net at IC3.4 (DRAIN1): now also M5.3 (-); no longer M5.4
- net at IC3.5 (DRAIN2): now also M5.4; no longer M5.2
- net at IC3.6 (DRAIN3): now also M5.2; no longer M5.3 (-)
- net at M8.2: now also IC4.14 (DRAIN7); no longer IC4.13 (DRAIN6)
- net at M8.3 (-): now also IC4.12 (DRAIN5); no longer IC4.14 (DRAIN7)
- net at M8.4: now also IC4.13 (DRAIN6); no longer IC4.12 (DRAIN5)
- net at M1.2: now also IC1.14 (DRAIN7); no longer IC1.13 (DRAIN6)
- net at M1.3 (-): now also IC1.12 (DRAIN5); no longer IC1.14 (DRAIN7)
- net at M1.4: now also IC1.13 (DRAIN6); no longer IC1.12 (DRAIN5)
- net at IC4.5 (DRAIN2): now also M7.4; no longer M7.2
- net at M7.3 (-): now also IC4.4 (DRAIN1); no longer IC4.6 (DRAIN3)
- net at M3.2: now also IC2.6 (DRAIN3); no longer IC2.5 (DRAIN2)
- net at M3.3 (-): now also IC2.4 (DRAIN1); no longer IC2.6 (DRAIN3)
- net at M3.4: now also IC2.5 (DRAIN2); no longer IC2.4 (DRAIN1)
- net at IC2.12 (DRAIN5): now also M4.3 (-); no longer M4.4
- net at IC2.13 (DRAIN6): now also M4.4; no longer M4.2
- net at IC2.14 (DRAIN7): now also M4.2; no longer M4.3 (-)
- net at M2.2: now also IC1.6 (DRAIN3); no longer IC1.5 (DRAIN2)
- net at M2.3 (-): now also IC1.4 (DRAIN1); no longer IC1.6 (DRAIN3)
- net at M2.4: now also IC1.5 (DRAIN2); no longer IC1.4 (DRAIN1)
- net +5VP renamed +12V
- net +12V: now also J2.3, M1.1, M2.1, M3.1, M4.1, M5.1, M6.1, M7.1, M8.1; no longer J1.1 (Pin_1), R1.1
- new net: IC4.6 (DRAIN3), M7.2
- no-connect marks 51 -> 50
Other:
- moved on the sheet: C9, M1, M2, M3, M4, M5, M6, M8, R9
